Commit message: added inertia

File: xacro/main.urdf (robot description, URDF)
Before this commit: robot arm_model, 6 links, 5 joints
Links:
- link base_link: mass None -> 1.0; geometry collision cylinder length=0.05 radius=0.1; visual cylinder length=0.05 radius=0.1
- link hand: mass None -> 1.0
- link lower_arm: mass None -> 1.0
- link torso: mass None -> 1.0
- link upper_arm: mass None -> 1.0

Commit message: collision and gazebo empty world

File: xacro/main.urdf (robot description, URDF)
Before this commit: robot arm_model, 6 links, 5 joints
Links:
- link hand: geometry collision box size=0.05 0.05 0.05; visual box size=0.05 0.05 0.05
- link lower_arm: geometry collision cylinder length=0.4 radius=0.05; visual cylinder length=0.4 radius=0.05
- link torso: geometry collision cylinder length=0.5 radius=0.05; visual cylinder length=0.5 radius=0.05
- link upper_arm: geometry collision cylinder length=0.4 radius=0.05; visual cylinder length=0.4 radius=0.05
