Commit message: new model of arm

File: arm_model/xacro/manipulator.urdf.xacro (robot description, xacro)
@@ -2,28 +2,28 @@
 <robot
 	xmlns:xacro="http://www.ros.org/wiki/xacro"
-	name="arm_model">
-	<xacro:macro name="arm_model">
+	name="manipulator_model">
+	<xacro:include filename="$(find arm_model)/xacro/macros.xacro" />
+	<xacro:macro name="manipulator_model">
 		<!--link name="world"/-->
 		<link name="arm_base_link">
 			<visual>
 				<geometry>
-					<cylinder length="0.05" radius="0.1"/>
+					<cylinder length="0.045" radius="0.055"/>
 				</geometry>
 				<material name="silver">
 					<color rgba="0.75 0.75 0.75 1"/>
 				</material>
-				<origin rpy="0 0 0" xyz="0 0 0.025"/>
-			</visual>
-			<collision>
-				<geometry>
-					<cylinder length="0.05" radius="0.1"/>
-				</geometry>
-				<origin rpy="0 0 0" xyz="0 0 0.025"/>
-			</collision>
-			<inertial>
-				<mass value="1.0"/>
-				<origin rpy="0 0 0" xyz="0 0 0.025"/>
-				<inertia ixx="0.0027" iyy="0.0027" izz="0.005"
-				ixy="0" ixz="0" iyz="0"/>
+				<origin rpy="0 0 0" xyz="0 0 0.0225"/>
+			</visual>
+			<collision>
+				<geometry>
+					<cylinder length="0.045" radius="0.055"/>
+				</geometry>
+				<origin rpy="0 0 0" xyz="0 0 0.0225"/>
+			</collision>
+			<inertial>
+				<mass value="1.0"/>
+				<origin rpy="0 0 0" xyz="0 0 0.0225"/>
+				<xacro:cylinder_inertia mass="1" r="0.055" l="0.05" />
 			</inertial>
 		</link>
@@ -32,110 +32,134 @@
 			<child link="arm_base_link"/>
 		</joint-->
-		<link name="torso">
-			<visual>
-				<geometry>
-					<cylinder length="0.5" radius="0.05"/>
+		<link name="turntable">
+			<visual>
+				<geometry>
+					<cylinder length="0.03" radius="0.055"/>
 				</geometry>
 				<material name="silver">
 					<color rgba="0.75 0.75 0.75 1"/>
 				</material>
-				<origin rpy="0 0 0" xyz="0 0 0.25"/>
-			</visual>
-			<collision>
-				<geometry>
-					<cylinder length="0.5" radius="0.05"/>
-				</geometry>
-				<origin rpy="0 0 0" xyz="0 0 0.25"/>
-			</collision>
-			<inertial>
-				<mass value="1.0"/>
-				<origin rpy="0 0 0" xyz="0 0 0.25"/>
-				<inertia ixx="0.02146" iyy="0.02146" izz="0.00125"
-				ixy="0" ixz="0" iyz="0"/>
-			</inertial>
-		</link>
-		<joint name="hip" type="continuous">
+				<origin rpy="0 0 0" xyz="0 0 0.015"/>
+			</visual>
+			<collision>
+				<geometry>
+					<cylinder length="0.03" radius="0.055"/>
+				</geometry>
+				<origin rpy="0 0 0" xyz="0 0 0.015"/>
+			</collision>
+			<inertial>
+				<mass value="1.0"/>
+				<origin rpy="0 0 0" xyz="0 0 0.015"/>
+				<xacro:cylinder_inertia mass="1" r="0.055" l="0.03" />
+			</inertial>
+		</link>
+		<joint name="turn" type="continuous">
 			<axis xyz="0 0 1"/>
 			<parent link="arm_base_link"/>
-			<child link="torso"/>
-			<origin rpy="0 0 0" xyz="0.0 0.0 0.05"/>
+			<child link="turntable"/>
+			<origin rpy="0 0 0" xyz="0.0 0.0 0.045"/>
 		</joint>
 		<link name="upper_arm">
 			<visual>
 				<geometry>
-					<cylinder length="0.4" radius="0.05"/>
-				</geometry>
-				<material name="silver"/>
-				<origin rpy="0 0 0" xyz="0 0 0.2"/>
-			</visual>
-			<collision>
-				<geometry>
-					<cylinder length="0.4" radius="0.05"/>
-				</geometry>
-				<origin rpy="0 0 0" xyz="0 0 0.2"/>
-			</collision>
-			<inertial>
-				<mass value="1.0"/>
-				<origin rpy="0 0 0" xyz="0 0 0.2"/>
-				<inertia ixx="0.01396" iyy="0.01396" izz="0.00125"
-				ixy="0" ixz="0" iyz="0"/>
+					<cylinder length="0.12" radius="0.0275"/>
+				</geometry>
+				<material name="silver"/>
+				<origin rpy="-1.5708 0 0" xyz="0 0.06 0"/>
+			</visual>
+			<collision>
+				<geometry>
+					<cylinder length="0.12" radius="0.0275"/>
+				</geometry>
+				<origin rpy="-1.5708 0 0" xyz="0 0.06 0"/>
+			</collision>
+			<inertial>
+				<mass value="1.0"/>
+				<origin rpy="-1.5708 0 0" xyz="0 0.06 0"/>
+				<xacro:cylinder_inertia mass="1" r="0.0275" l="0.12" />
 			</inertial>
 		</link>
 		<joint name="shoulder" type="continuous">
-			<axis xyz="0 1 0"/>
-			<parent link="torso"/>
+			<axis xyz="0 0 1"/>
+			<parent link="turntable"/>
 			<child link="upper_arm"/>
-			<origin rpy="0 1.5708 0" xyz="0.0 -0.1 0.45"/>
+			<origin rpy="1.5708 0 0" xyz="0.0 0.0 0.03"/>
+		</joint>
+		<link name="middle_arm">
+			<visual>
+				<geometry>
+					<cylinder length="0.12" radius="0.0275"/>
+				</geometry>
+				<material name="silver"/>
+				<origin rpy="-1.5708 0 0" xyz="0 0.06 0"/>
+			</visual>
+			<collision>
+				<geometry>
+					<cylinder length="0.12" radius="0.0275"/>
+				</geometry>
+				<origin rpy="-1.5708 0 0" xyz="0 0.06 0"/>
+			</collision>
+			<inertial>
+				<mass value="1.0"/>
+				<origin rpy="-1.5708 0 0" xyz="0 0.06 0"/>
+				<xacro:cylinder_inertia mass="1" r="0.0275" l="0.12" />
+			</inertial>
+		</link>
+		<joint name="elbow" type="continuous">
+			<axis xyz="0 0 1"/>
+			<parent link="upper_arm"/>
+			<child link="middle_arm"/>
+			<origin rpy="0 0 0" xyz="0 0.12 0"/>
 		</joint>
 		<link name="lower_arm">
 			<visual>
 				<geometry>
-					<cylinder length="0.4" radius="0.05"/>
-				</geometry>
-				<material name="silver"/>
-				<origin rpy="0 0 0" xyz="0 0 0.2"/>
-			</visual>
-			<collision>
-				<geometry>
-					<cylinder length="0.4" radius="0.05"/>
-				</geometry>
-				<origin rpy="0 0 0" xyz="0 0 0.2"/>
-			</collision>
-			<inertial>
-				<mass value="1.0"/>
-				<origin rpy="0 0 0" xyz="0 0 0.2"/>
-				<inertia ixx="0.01396" iyy="0.01396" izz="0.00125"
-				ixy="0" ixz="0" iyz="0"/>
-			</inertial>
-		</link>
-		<joint name="elbow" type="continuous">
-			<axis xyz="0 1 0"/>
-			<parent link="upper_arm"/>
+					<cylinder length="0.055" radius="0.0275"/>
+				</geometry>
+				<material name="silver"/>
+				<origin rpy="-1.5708 0 0" xyz="0 0.0275 0"/>
+			</visual>
+			<collision>
+				<geometry>
+					<cylinder length="0.055" radius="0.0275"/>
+				</geometry>
+				<origin rpy="-1.5708 0 0" xyz="0 0.0275 0"/>
+			</collision>
+			<inertial>
+				<mass value="1.0"/>
+				<origin rpy="-1.5708 0 0" xyz="0 0.0275 0"/>
+				<xacro:cylinder_inertia mass="1" r="0.0275" l="0.055" />
+			</inertial>
+		</link>
+		<joint name="another_elbow" type="continuous">
+			<axis xyz="0 0 1"/>
+			<parent link="middle_arm"/>
 			<child link="lower_arm"/>
-			<origin rpy="0 0 0" xyz="0.0 0.1 0.35"/>
+			<origin rpy="0 0 0" xyz="0 0.12 0"/>
 		</joint>
 		<link name="hand">
 			<visual>
 				<geometry>
-					<box size="0.05 0.05 0.05"/>
-				</geometry>
-				<material name="silver"/>
-			</visual>
-			<collision>
-				<geometry>
-					<box size="0.05 0.05 0.05"/>
-				</geometry>
-			</collision>
-			<inertial>
-				<mass value="1.0"/>
-				<inertia ixx="0.00042" iyy="0.00042" izz="0.00042"
-				ixy="0" ixz="0" iyz="0"/>
-			</inertial>
-		</link>
-		<joint name="wrist" type="continuous">
-			<axis xyz="0 1 0"/>
+					<box size="0.03 0.03 0.03"/>
+				</geometry>
+				<material name="silver"/>
+				<origin rpy="0 0 0" xyz="0 0 0.015"/>
+			</visual>
+			<collision>
+				<geometry>
+					<box size="0.03 0.03 0.03"/>
+				</geometry>
+				<origin rpy="0 0 0" xyz="0 0 0.015"/>
+			</collision>
+			<inertial>
+				<mass value="1.0"/>
+				<origin rpy="0 0 0" xyz="0 0 0.015"/>
+				<xacro:box_inertia mass="1" x="0.03" y="0.03" z="0.03" />
+			</inertial>
+		</link>
+		<joint name="wrist" type="fixed">
 			<parent link="lower_arm"/>
 			<child link="hand"/>
-			<origin rpy="0 0 0" xyz="0.0 0.0 0.425"/>
+			<origin rpy="-1.5708 0 0" xyz="0.0 0.055 0.0"/>
 		</joint>
 		<!--Transmission Descriptions-->
@@ -190,3 +214,4 @@
 		</gazebo>
 	</xacro:macro>
+	<xacro:manipulator_model/>
 </robot>

Commit message: movit of our manipulator, planning but not executing

File: arm_model/xacro/manipulator.urdf.xacro (robot description, xacro)
@@ -5,6 +5,6 @@
 	<xacro:include filename="$(find arm_model)/xacro/macros.xacro" />
 	<xacro:macro name="manipulator_model">
-		<!--link name="world"/-->
-		<link name="arm_base_link">
+		<link name="world"/>
+		<link name="manipulator_base_link">
 			<visual>
 				<geometry>
@@ -28,8 +28,9 @@
 			</inertial>
 		</link>
-		<!--joint name="fixed" type="fixed">
+		<joint name="planar" type="fixed">
+			<!--axis xyz="0 0 1"/-->
 			<parent link="world"/>
-			<child link="arm_base_link"/>
-		</joint-->
+			<child link="manipulator_base_link"/>
+		</joint>
 		<link name="turntable">
 			<visual>
@@ -56,5 +57,5 @@
 		<joint name="turn" type="continuous">
 			<axis xyz="0 0 1"/>
-			<parent link="arm_base_link"/>
+			<parent link="manipulator_base_link"/>
 			<child link="turntable"/>
 			<origin rpy="0 0 0" xyz="0.0 0.0 0.045"/>
@@ -84,5 +85,5 @@
 			<parent link="turntable"/>
 			<child link="upper_arm"/>
-			<origin rpy="1.5708 0 0" xyz="0.0 0.0 0.03"/>
+			<origin rpy="1.5708 0 0" xyz="0.0 0.0 0.0575"/>
 		</joint>
 		<link name="middle_arm">
@@ -92,15 +93,15 @@
 				</geometry>
 				<material name="silver"/>
-				<origin rpy="-1.5708 0 0" xyz="0 0.06 0"/>
-			</visual>
-			<collision>
-				<geometry>
-					<cylinder length="0.12" radius="0.0275"/>
-				</geometry>
-				<origin rpy="-1.5708 0 0" xyz="0 0.06 0"/>
-			</collision>
-			<inertial>
-				<mass value="1.0"/>
-				<origin rpy="-1.5708 0 0" xyz="0 0.06 0"/>
+				<origin rpy="-1.5708 0 0" xyz="0 0.06 0.0555"/>
+			</visual>
+			<collision>
+				<geometry>
+					<cylinder length="0.12" radius="0.0275"/>
+				</geometry>
+				<origin rpy="-1.5708 0 0" xyz="0 0.06 0.0555"/>
+			</collision>
+			<inertial>
+				<mass value="1.0"/>
+				<origin rpy="-1.5708 0 0" xyz="0 0.06 0.0555"/>
 				<xacro:cylinder_inertia mass="1" r="0.0275" l="0.12" />
 			</inertial>
@@ -166,5 +167,5 @@
 		<transmission name="tran0">
 			<type>transmission_interface/SimpleTransmission</type>
-			<joint name="hip">
+			<joint name="turn">
 				<hardwareInterface>PositionJointInterface</hardwareInterface>
 			</joint>
@@ -196,5 +197,5 @@
 		<transmission name="tran3">
 			<type>transmission_interface/SimpleTransmission</type>
-			<joint name="wrist">
+			<joint name="another_elbow">
 				<hardwareInterface>PositionJointInterface</hardwareInterface>
 			</joint>
@@ -210,5 +211,5 @@
 			<!-- joint_state_publisher plugin -->
 			<plugin name="joint_state_publisher" filename="libgazebo_ros_joint_state_publisher.so">
-					<jointName>hip, shoulder, elbow, wrist</jointName>
+					<jointName>turn, shoulder, elbow, another_elbow</jointName>
 			</plugin>
 		</gazebo>

Commit message: mobile base using 2 prismatic joints

File: arm_model/xacro/manipulator.urdf.xacro (robot description, xacro)
@@ -6,4 +6,24 @@
 	<xacro:macro name="manipulator_model">
 		<link name="world"/>
+		<joint name="move_x" type="prismatic">
+			<axis xyz="1 0 0"/>
+			<parent link="world"/>
+			<child link="x_axis_moving_base"/>
+			<limit effort="1000.0" lower="-1" upper="1" velocity="0.5"/>
+			<origin rpy="0 0 0" xyz="0.0 0.0 0.0"/>
+		</joint>
+		<link name="x_axis_moving_base"/>
+		<joint name="move_y" type="prismatic">
+			<axis xyz="0 1 0"/>
+			<parent link="x_axis_moving_base"/>
+			<child link="y_axis_moving_base"/>
+			<limit effort="1000.0" lower="-1" upper="1" velocity="0.5"/>
+			<origin rpy="0 0 0" xyz="0.0 0.0 0.0"/>
+		</joint>
+		<link name="y_axis_moving_base"/>
+		<joint name="planar" type="fixed">
+			<parent link="y_axis_moving_base"/>
+			<child link="manipulator_base_link"/>
+		</joint>
 		<link name="manipulator_base_link">
 			<visual>
@@ -28,9 +48,4 @@
 			</inertial>
 		</link>
-		<joint name="planar" type="fixed">
-			<!--axis xyz="0 0 1"/-->
-			<parent link="world"/>
-			<child link="manipulator_base_link"/>
-		</joint>
 		<link name="turntable">
 			<visual>
@@ -205,11 +220,31 @@
 			</actuator>
 		</transmission>
+		<transmission name="tran4">
+			<type>transmission_interface/SimpleTransmission</type>
+			<joint name="move_x">
+				<hardwareInterface>EffortJointInterface</hardwareInterface>
+			</joint>
+			<actuator name="motor4">
+				<hardwareInterface>EffortJointInterface</hardwareInterface>
+				<mechanicalReduction>1</mechanicalReduction>
+			</actuator>
+		</transmission>
+		<transmission name="tran5">
+			<type>transmission_interface/SimpleTransmission</type>
+			<joint name="move_y">
+				<hardwareInterface>EffortJointInterface</hardwareInterface>
+			</joint>
+			<actuator name="motor5">
+				<hardwareInterface>EffortJointInterface</hardwareInterface>
+				<mechanicalReduction>1</mechanicalReduction>
+			</actuator>
+		</transmission>
 		<!-- Gazebo Plugins -->
 		<gazebo>
-			<!--ros_control plugin-->
+			<!-- ros_control plugin -->
 			<plugin name="control" filename="libgazebo_ros_control.so"/>
 			<!-- joint_state_publisher plugin -->
 			<plugin name="joint_state_publisher" filename="libgazebo_ros_joint_state_publisher.so">
-					<jointName>turn, shoulder, elbow, another_elbow</jointName>
+					<jointName>turn, shoulder, elbow, another_elbow, move_y, move_x</jointName>
 			</plugin>
 		</gazebo>

Commit message: mobile base running

File: arm_model/xacro/manipulator.urdf.xacro (robot description, xacro)
@@ -13,5 +13,11 @@
 			<origin rpy="0 0 0" xyz="0.0 0.0 0.0"/>
 		</joint>
-		<link name="x_axis_moving_base"/>
+		<link name="x_axis_moving_base">
+			<inertial>
+				<mass value="1.0"/>
+				<origin rpy="0 0 0" xyz="0 0 0.0225"/>
+				<xacro:cylinder_inertia mass="1" r="0.055" l="0.05" />
+			</inertial>
+		</link>
 		<joint name="move_y" type="prismatic">
 			<axis xyz="0 1 0"/>
@@ -21,5 +27,11 @@
 			<origin rpy="0 0 0" xyz="0.0 0.0 0.0"/>
 		</joint>
-		<link name="y_axis_moving_base"/>
+		<link name="y_axis_moving_base">
+			<inertial>
+				<mass value="1.0"/>
+				<origin rpy="0 0 0" xyz="0 0 0.0225"/>
+				<xacro:cylinder_inertia mass="1" r="0.055" l="0.05" />
+			</inertial>
+		</link>
 		<joint name="planar" type="fixed">
 			<parent link="y_axis_moving_base"/>
@@ -223,8 +235,8 @@
 			<type>transmission_interface/SimpleTransmission</type>
 			<joint name="move_x">
-				<hardwareInterface>EffortJointInterface</hardwareInterface>
+				<hardwareInterface>PositionJointInterface</hardwareInterface>
 			</joint>
 			<actuator name="motor4">
-				<hardwareInterface>EffortJointInterface</hardwareInterface>
+				<hardwareInterface>PositionJointInterface</hardwareInterface>
 				<mechanicalReduction>1</mechanicalReduction>
 			</actuator>
@@ -233,8 +245,8 @@
 			<type>transmission_interface/SimpleTransmission</type>
 			<joint name="move_y">
-				<hardwareInterface>EffortJointInterface</hardwareInterface>
+				<hardwareInterface>PositionJointInterface</hardwareInterface>
 			</joint>
 			<actuator name="motor5">
-				<hardwareInterface>EffortJointInterface</hardwareInterface>
+				<hardwareInterface>PositionJointInterface</hardwareInterface>
 				<mechanicalReduction>1</mechanicalReduction>
 			</actuator>
@@ -246,5 +258,5 @@
 			<!-- joint_state_publisher plugin -->
 			<plugin name="joint_state_publisher" filename="libgazebo_ros_joint_state_publisher.so">
-					<jointName>turn, shoulder, elbow, another_elbow, move_y, move_x</jointName>
+					<jointName>turn, shoulder, elbow, another_elbow, move_x, move_y</jointName>
 			</plugin>
 		</gazebo>

Commit message: model with y-axis constraint

File: arm_model/xacro/manipulator.urdf.xacro (robot description, xacro)
@@ -6,34 +6,33 @@
 	<xacro:macro name="manipulator_model">
 		<link name="world"/>
-		<joint name="move_x" type="prismatic">
+		<link name="rotate_moving_base">
+			<inertial>
+				<mass value="1.0"/>
+				<origin rpy="0 0 0" xyz="0 0 0.0225"/>
+				<xacro:cylinder_inertia mass="1" r="0.055" l="0.05" />
+			</inertial>
+		</link>
+		<joint name="move_rotate" type="continuous">
+			<axis xyz="0 0 1"/>
+			<parent link="world"/>
+			<child link="rotate_moving_base"/>
+			<origin rpy="0 0 0" xyz="0.0 0.0 0.0"/>
+		</joint>
+		<link name="forward_moving_base">
+			<inertial>
+				<mass value="1.0"/>
+				<origin rpy="0 0 0" xyz="0 0 0.0225"/>
+				<xacro:cylinder_inertia mass="1" r="0.055" l="0.05" />
+			</inertial>
+		</link>
+		<joint name="move_forward" type="prismatic">
 			<axis xyz="1 0 0"/>
-			<parent link="world"/>
-			<child link="x_axis_moving_base"/>
+			<parent link="rotate_moving_base"/>
+			<child link="forward_moving_base"/>
 			<limit effort="1000.0" lower="-1" upper="1" velocity="0.5"/>
 			<origin rpy="0 0 0" xyz="0.0 0.0 0.0"/>
 		</joint>
-		<link name="x_axis_moving_base">
-			<inertial>
-				<mass value="1.0"/>
-				<origin rpy="0 0 0" xyz="0 0 0.0225"/>
-				<xacro:cylinder_inertia mass="1" r="0.055" l="0.05" />
-			</inertial>
-		</link>
-		<joint name="move_y" type="prismatic">
-			<axis xyz="0 1 0"/>
-			<parent link="x_axis_moving_base"/>
-			<child link="y_axis_moving_base"/>
-			<limit effort="1000.0" lower="-1" upper="1" velocity="0.5"/>
-			<origin rpy="0 0 0" xyz="0.0 0.0 0.0"/>
-		</joint>
-		<link name="y_axis_moving_base">
-			<inertial>
-				<mass value="1.0"/>
-				<origin rpy="0 0 0" xyz="0 0 0.0225"/>
-				<xacro:cylinder_inertia mass="1" r="0.055" l="0.05" />
-			</inertial>
-		</link>
-		<joint name="planar" type="fixed">
-			<parent link="y_axis_moving_base"/>
+		<joint name="fixed" type="fixed">
+			<parent link="forward_moving_base"/>
 			<child link="manipulator_base_link"/>
 		</joint>
@@ -41,5 +40,5 @@
 			<visual>
 				<geometry>
-					<cylinder length="0.045" radius="0.055"/>
+					<cylinder length="0.045" radius="0.1"/>
 				</geometry>
 				<material name="silver">
@@ -50,12 +49,12 @@
 			<collision>
 				<geometry>
-					<cylinder length="0.045" radius="0.055"/>
-				</geometry>
-				<origin rpy="0 0 0" xyz="0 0 0.0225"/>
-			</collision>
-			<inertial>
-				<mass value="1.0"/>
-				<origin rpy="0 0 0" xyz="0 0 0.0225"/>
-				<xacro:cylinder_inertia mass="1" r="0.055" l="0.05" />
+					<cylinder length="0.045" radius="0.1"/>
+				</geometry>
+				<origin rpy="0 0 0" xyz="0 0 0.0225"/>
+			</collision>
+			<inertial>
+				<mass value="1.0"/>
+				<origin rpy="0 0 0" xyz="0 0 0.0225"/>
+				<xacro:cylinder_inertia mass="1" r="0.1" l="0.05" />
 			</inertial>
 		</link>
@@ -234,5 +233,5 @@
 		<transmission name="tran4">
 			<type>transmission_interface/SimpleTransmission</type>
-			<joint name="move_x">
+			<joint name="move_rotate">
 				<hardwareInterface>PositionJointInterface</hardwareInterface>
 			</joint>
@@ -244,5 +243,5 @@
 		<transmission name="tran5">
 			<type>transmission_interface/SimpleTransmission</type>
-			<joint name="move_y">
+			<joint name="move_forward">
 				<hardwareInterface>PositionJointInterface</hardwareInterface>
 			</joint>
@@ -258,5 +257,5 @@
 			<!-- joint_state_publisher plugin -->
 			<plugin name="joint_state_publisher" filename="libgazebo_ros_joint_state_publisher.so">
-					<jointName>turn, shoulder, elbow, another_elbow, move_x, move_y</jointName>
+					<jointName>turn, shoulder, elbow, another_elbow, move_rotate, move_forward</jointName>
 			</plugin>
 		</gazebo>
