Commit message: velocity transmissions implemented

File: manipulator_model/xacro/manipulator_velocity.urdf.xacro (robot description, xacro)
@@ -192,10 +192,10 @@
 		</joint>
 		<!--Transmission Descriptions-->
-		<xacro:effort_transmission name="tran0" joint="turn" actuator="motor0"/>
-		<xacro:effort_transmission name="tran1" joint="shoulder" actuator="motor1"/>
-		<xacro:effort_transmission name="tran2" joint="elbow" actuator="motor2"/>
-		<xacro:effort_transmission name="tran3" joint="another_elbow" actuator="motor3"/>
-		<xacro:effort_transmission name="tran4" joint="move_rotate" actuator="motor4"/>
-		<xacro:effort_transmission name="tran5" joint="move_forward" actuator="motor5"/>
+		<xacro:velocity_transmission name="tran0" joint="turn" actuator="motor0"/>
+		<xacro:velocity_transmission name="tran1" joint="shoulder" actuator="motor1"/>
+		<xacro:velocity_transmission name="tran2" joint="elbow" actuator="motor2"/>
+		<xacro:velocity_transmission name="tran3" joint="another_elbow" actuator="motor3"/>
+		<xacro:velocity_transmission name="tran4" joint="move_rotate" actuator="motor4"/>
+		<xacro:velocity_transmission name="tran5" joint="move_forward" actuator="motor5"/>
 		<!-- Gazebo Plugins -->
 		<gazebo>

File: manipulator_model/xacro/transmission_macros.xacro (robot description, xacro)
@@ -1,12 +1,12 @@
 <?xml version="1.0"?>
 <robot xmlns:xacro="http://www.ros.org/wiki/xacro">
-    <xacro:macro name="effort_transmission" params="name joint actuator">
+    <xacro:macro name="velocity_transmission" params="name joint actuator">
       <transmission name="${name}">
         <type>transmission_interface/SimpleTransmission</type>
         <joint name="${joint}">
-          <hardwareInterface>hardware_interface/EffortJointInterface</hardwareInterface>
+          <hardwareInterface>hardware_interface/VelocityJointInterface</hardwareInterface>
         </joint>
         <actuator name="${actuator}">
-          <hardwareInterface>hardware_interface/EffortJointInterface</hardwareInterface>
+          <hardwareInterface>hardware_interface/VelocityJointInterface</hardwareInterface>
           <mechanicalReduction>1</mechanicalReduction>
         </actuator>
