Commit message: added xacro for transmission

File: manipulator_model/xacro/manipulator.urdf.xacro (robot description, xacro)
@@ -3,5 +3,6 @@
 	xmlns:xacro="http://www.ros.org/wiki/xacro"
 	name="manipulator_model">
-	<xacro:include filename="$(find manipulator_model)/xacro/macros.xacro" />
+	<xacro:include filename="$(find manipulator_model)/xacro/inertia_macros.xacro" />
+	<xacro:include filename="$(find manipulator_model)/xacro/transmission_macros.xacro" />
 	<xacro:macro name="manipulator_model">
 		<link name="world"/>
@@ -191,64 +192,10 @@
 		</joint>
 		<!--Transmission Descriptions-->
-		<transmission name="tran0">
-			<type>transmission_interface/SimpleTransmission</type>
-			<joint name="turn">
-				<hardwareInterface>PositionJointInterface</hardwareInterface>
-			</joint>
-			<actuator name="motor0">
-				<hardwareInterface>PositionJointInterface</hardwareInterface>
-				<mechanicalReduction>1</mechanicalReduction>
-			</actuator>
-		</transmission>
-		<transmission name="tran1">
-			<type>transmission_interface/SimpleTransmission</type>
-			<joint name="shoulder">
-				<hardwareInterface>PositionJointInterface</hardwareInterface>
-			</joint>
-			<actuator name="motor1">
-				<hardwareInterface>PositionJointInterface</hardwareInterface>
-				<mechanicalReduction>1</mechanicalReduction>
-			</actuator>
-		</transmission>
-		<transmission name="tran2">
-			<type>transmission_interface/SimpleTransmission</type>
-			<joint name="elbow">
-				<hardwareInterface>PositionJointInterface</hardwareInterface>
-			</joint>
-			<actuator name="motor2">
-				<hardwareInterface>PositionJointInterface</hardwareInterface>
-				<mechanicalReduction>1</mechanicalReduction>
-			</actuator>
-		</transmission>
-		<transmission name="tran3">
-			<type>transmission_interface/SimpleTransmission</type>
-			<joint name="another_elbow">
-				<hardwareInterface>PositionJointInterface</hardwareInterface>
-			</joint>
-			<actuator name="motor3">
-				<hardwareInterface>PositionJointInterface</hardwareInterface>
-				<mechanicalReduction>1</mechanicalReduction>
-			</actuator>
-		</transmission>
-		<transmission name="tran4">
-			<type>transmission_interface/SimpleTransmission</type>
-			<joint name="move_rotate">
-				<hardwareInterface>PositionJointInterface</hardwareInterface>
-			</joint>
-			<actuator name="motor4">
-				<hardwareInterface>PositionJointInterface</hardwareInterface>
-				<mechanicalReduction>1</mechanicalReduction>
-			</actuator>
-		</transmission>
-		<transmission name="tran5">
-			<type>transmission_interface/SimpleTransmission</type>
-			<joint name="move_forward">
-				<hardwareInterface>PositionJointInterface</hardwareInterface>
-			</joint>
-			<actuator name="motor5">
-				<hardwareInterface>PositionJointInterface</hardwareInterface>
-				<mechanicalReduction>1</mechanicalReduction>
-			</actuator>
-		</transmission>
+		<xacro:position_transmission name="tran0" joint="turn" actuator="motor0"/>
+		<xacro:position_transmission name="tran1" joint="shoulder" actuator="motor1"/>
+		<xacro:position_transmission name="tran2" joint="elbow" actuator="motor2"/>
+		<xacro:position_transmission name="tran3" joint="another_elbow" actuator="motor3"/>
+		<xacro:position_transmission name="tran4" joint="move_rotate" actuator="motor4"/>
+		<xacro:position_transmission name="tran5" joint="move_forward" actuator="motor5"/>
 		<!-- Gazebo Plugins -->
 		<gazebo>

Commit message: kobuki measures added

File: manipulator_model/xacro/manipulator.urdf.xacro (robot description, xacro)
@@ -10,5 +10,5 @@
 			<inertial>
 				<mass value="1.0"/>
-				<origin rpy="0 0 0" xyz="0 0 0.0225"/>
+				<origin rpy="0 0 0" xyz="0 0 0.0625"/>
 				<xacro:cylinder_inertia mass="1" r="0.055" l="0.05" />
 			</inertial>
@@ -23,5 +23,5 @@
 			<inertial>
 				<mass value="1.0"/>
-				<origin rpy="0 0 0" xyz="0 0 0.0225"/>
+				<origin rpy="0 0 0" xyz="0 0 0.0625"/>
 				<xacro:cylinder_inertia mass="1" r="0.055" l="0.05" />
 			</inertial>
@@ -41,20 +41,20 @@
 			<visual>
 				<geometry>
-					<cylinder length="0.045" radius="0.1"/>
+					<cylinder length="0.125" radius="0.175"/>
 				</geometry>
 				<material name="silver">
 					<color rgba="0.75 0.75 0.75 1"/>
 				</material>
-				<origin rpy="0 0 0" xyz="0 0 0.0225"/>
-			</visual>
-			<collision>
-				<geometry>
-					<cylinder length="0.045" radius="0.1"/>
-				</geometry>
-				<origin rpy="0 0 0" xyz="0 0 0.0225"/>
-			</collision>
-			<inertial>
-				<mass value="1.0"/>
-				<origin rpy="0 0 0" xyz="0 0 0.0225"/>
+				<origin rpy="0 0 0" xyz="0 0 0.0625"/>
+			</visual>
+			<collision>
+				<geometry>
+					<cylinder length="0.125" radius="0.175"/>
+				</geometry>
+				<origin rpy="0 0 0" xyz="0 0 0.0625"/>
+			</collision>
+			<inertial>
+				<mass value="1.0"/>
+				<origin rpy="0 0 0" xyz="0 0 0.0625"/>
 				<xacro:cylinder_inertia mass="1" r="0.1" l="0.05" />
 			</inertial>
@@ -86,5 +86,5 @@
 			<parent link="manipulator_base_link"/>
 			<child link="turntable"/>
-			<origin rpy="0 0 0" xyz="0.0 0.0 0.045"/>
+			<origin rpy="0 0 0" xyz="0.0 0.0 0.125"/>
 		</joint>
 		<link name="upper_arm">

Commit message: changes in contorller and desired joint trajectory

File: manipulator_model/xacro/manipulator.urdf.xacro (robot description, xacro)
@@ -192,10 +192,10 @@
 		</joint>
 		<!--Transmission Descriptions-->
-		<xacro:position_transmission name="tran0" joint="turn" actuator="motor0"/>
-		<xacro:position_transmission name="tran1" joint="shoulder" actuator="motor1"/>
-		<xacro:position_transmission name="tran2" joint="elbow" actuator="motor2"/>
-		<xacro:position_transmission name="tran3" joint="another_elbow" actuator="motor3"/>
-		<xacro:position_transmission name="tran4" joint="move_rotate" actuator="motor4"/>
-		<xacro:position_transmission name="tran5" joint="move_forward" actuator="motor5"/>
+		<xacro:effort_transmission name="tran0" joint="turn" actuator="motor0"/>
+		<xacro:effort_transmission name="tran1" joint="shoulder" actuator="motor1"/>
+		<xacro:effort_transmission name="tran2" joint="elbow" actuator="motor2"/>
+		<xacro:effort_transmission name="tran3" joint="another_elbow" actuator="motor3"/>
+		<xacro:effort_transmission name="tran4" joint="move_rotate" actuator="motor4"/>
+		<xacro:effort_transmission name="tran5" joint="move_forward" actuator="motor5"/>
 		<!-- Gazebo Plugins -->
 		<gazebo>

File: manipulator_model/xacro/transmission_macros.xacro (robot description, xacro)
@@ -1,12 +1,12 @@
 <?xml version="1.0"?>
 <robot xmlns:xacro="http://www.ros.org/wiki/xacro">
-    <xacro:macro name="velocity_transmission" params="name joint actuator">
+    <xacro:macro name="effort_transmission" params="name joint actuator">
       <transmission name="${name}">
         <type>transmission_interface/SimpleTransmission</type>
         <joint name="${joint}">
-          <hardwareInterface>hardware_interface/VelocityJointInterface</hardwareInterface>
+          <hardwareInterface>hardware_interface/EffortJointInterface</hardwareInterface>
         </joint>
         <actuator name="${actuator}">
-          <hardwareInterface>hardware_interface/VelocityJointInterface</hardwareInterface>
+          <hardwareInterface>hardware_interface/EffortJointInterface</hardwareInterface>
           <mechanicalReduction>1</mechanicalReduction>
         </actuator>
